File: power_board/power_board.kicad_pcb (KiCad board)
At the start: 2 copper layers, 60 x 60 mm, 23 parts, among them J1 Screw_Terminal_01x02, J2 Screw_Terminal_01x03, J3 Conn_01x12, U1 LM7805_TO220, U2 LM7805_TO220, U3 LM7805_TO220

Commit message: update pcb
Parts:
- moved J1 36.7 mm to (131.4, 121.6), turned to -45 degrees
- moved J2 35.2 mm to (137.6, 83.4), turned to -135 degrees
- moved U1 34.6 mm to (141.3, 119.5), turned to -90 degrees
- moved C1 31.6 mm to (163.0, 125.0), turned to 90 degrees
- moved J3 29.7 mm to (172.5, 120.7), turned to 180 degrees
- moved C4 29.5 mm to (163.1, 118.6), turned to -90 degrees
- moved C3 19.1 mm to (146.8, 102.6)
- moved C10 14.3 mm to (150.9, 94.4)
- moved C6 14.3 mm to (151.0, 100.4)
- moved C8 14.3 mm to (151.0, 97.4)
- moved R2 14.3 mm to (154.0, 99.4)
- moved R3 14.3 mm to (154.0, 95.4)
- moved C9 14.0 mm to (162.8, 94.6)
- moved C5 14.0 mm to (162.8, 100.6)
- moved C7 14.0 mm to (162.8, 97.6)
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Routing:
- net -5V: track 8.17 -> 47.8 mm
- net GND: track 57.0 -> 22.4 mm, vias 1 -> 0
- net +Batt1: track 15.3 -> 43.9 mm
- net -Batt2: track 52.5 -> 28.9 mm
- net +3V3: track 20.1 -> 36.4 mm
- net +BATT: track 31.6 -> 47.5 mm
- net +5VA: track 13.9 -> 23.7 mm
- net +Batt2: track 12.5 -> 16.6 mm
- net Net-(C6-Pad2): track 17.6 -> 14.4 mm
- net Net-(C5-Pad1): track 26.7 -> 28.6 mm, vias 0 -> 3
- added copper zone on F.Cu, net GND
