File: uc_board/uc_board/uc_board.kicad_pcb (KiCad board)
At the start: 2 copper layers, 60 x 60 mm, 5 parts, among them J1 Conn_01x12

Commit message: update pcb
Parts:
- moved A1 40.7 mm to (139.9, 84.0), turned to 0 degrees
Routing:
- net DRDY: track 35.0 -> 13.5 mm
- net Rx: track 47.8 -> 41.7 mm
- net +3V3: track 41.3 -> 35.5 mm

Commit message: update pcb
Parts:
- turned J1 to 180 degrees
Connections:
- J1 pad 12: unconnected-(J1-Pad12) -> GNDA
- J1 pad 3: unconnected-(J1-Pad3) -> +5VA
- J1 pad 4: unconnected-(J1-Pad4) -> -5VA
- J1 pad 8: Tx -> Rx
- J1 pad 9: Rx -> Tx
Routing:
- net Rx: track 41.7 -> 46.5 mm
- net Tx: track 37.0 -> 41.2 mm
- net DRDY: track 13.5 -> 12.4 mm
Changed lines of the file:
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@@
   (net 26 "unconnected-(A1-Pad27)")
   (net 27 "unconnected-(A1-Pad28)")
-  (net 28 "unconnected-(J1-Pad3)")
-  (net 29 "unconnected-(J1-Pad4)")
+  (net 28 "+5VA")
+  (net 29 "-5VA")
   (net 30 "unconnected-(J1-Pad5)")
   (net 31 "unconnected-(J1-Pad7)")
   (net 32 "unconnected-(J1-Pad10)")
   (net 33 "unconnected-(J1-Pad11)")
-  (net 34 "unconnected-(J1-Pad12)")
+  (net 34 "GNDA")
   (footprint "Module:Adafruit_Feather" (layer "F.Cu")
     (at 139.9475 83.95)
@@
   )
   (footprint "Connector_PinSocket_2.54mm:PinSocket_1x12_P2.54mm_Vertical" (layer "F.Cu")
-    (at 172.479 104.99)
+    (at 172.479 104.99 180)
     (descr "Through hole straight socket strip, 1x12, 2.54mm pitch, single row (from Kicad 4.0.7), script generated")
     (tags "Through hole socket strip THT 1x12 2.54mm single row")
@@
     (fp_line (start 1.295 -14.585) (end 1.295 15.26) (layer "F.Fab") (width 0.1))
     (fp_line (start 1.295 15.26) (end -1.245 15.26) (layer "F.Fab") (width 0.1))
-    (pad "1" thru_hole rect (at 0.025 -13.95) (size 1.7 1.7) (drill 1) (layers *.Cu *.Mask)
+    (pad "1" thru_hole rect (at 0.025 -13.95 180) (size 1.7 1.7) (drill 1) (layers *.Cu *.Mask)
       (net 4 "GND") (pinfunction "Pin_1") (pintype "passive"))
-    (pad "2" thru_hole oval (at 0.025 -11.41) (size 1.7 1.7) (drill 1) (layers *.Cu *.Mask)
+    (pad "2" thru_hole oval (at 0.025 -11.41 180) (size 1.7 1.7) (drill 1) (layers *.Cu *.Mask)
       (net 2 "+3V3") (pinfunction "Pin_2") (pintype "passive"))
-    (pad "3" thru_hole oval (at 0.025 -8.87) (size 1.7 1.7) (drill 1) (layers *.Cu *.Mask)
-      (net 28 "unconnected-(J1-Pad3)") (pinfunction "Pin_3") (pintype "passive+no_connect"))
-    (pad "4" thru_hole oval (at 0.025 -6.33) (size 1.7 1.7) (drill 1) (layers *.Cu *.Mask)
-      (net 29 "unconnected-(J1-Pad4)") (pinfunction "Pin_4") (pintype "passive+no_connect"))
-    (pad "5" thru_hole oval (at 0.025 -3.79) (size 1.7 1.7) (drill 1) (layers *.Cu *.Mask)
+    (pad "3" thru_hole oval (at 0.025 -8.87 180) (size 1.7 1.7) (drill 1) (layers *.Cu *.Mask)
+      (net 28 "+5VA") (pinfunction "Pin_3") (pintype "passive"))
+    (pad "4" thru_hole oval (at 0.025 -6.33 180) (size 1.7 1.7) (drill 1) (layers *.Cu *.Mask)
+      (net 29 "-5VA") (pinfunction "Pin_4") (pintype "passive"))
+    (pad "5" thru_hole oval (at 0.025 -3.79 180) (size 1.7 1.7) (drill 1) (layers *.Cu *.Mask)
       (net 30 "unconnected-(J1-Pad5)") (pinfunction "Pin_5") (pintype "passive+no_connect"))
-    (pad "6" thru_hole oval (at 0.025 -1.25) (size 1.7 1.7) (drill 1) (layers *.Cu *.Mask)
+    (pad "6" thru_hole oval (at 0.025 -1.25 180) (size 1.7 1.7) (drill 1) (layers *.Cu *.Mask)
       (net 22 "DRDY") (pinfunction "Pin_6") (pintype "passive"))
-    (pad "7" thru_hole oval (at 0.025 1.29) (size 1.7 1.7) (drill 1) (layers *.Cu *.Mask)
+    (pad "7" thru_hole oval (at 0.025 1.29 180) (size 1.7 1.7) (drill 1) (layers *.Cu *.Mask)
       (net 31 "unconnected-(J1-Pad7)") (pinfunction "Pin_7") (pintype "passive+no_connect"))
-    (pad "8" thru_hole oval (at 0.025 3.83) (size 1.7 1.7) (drill 1) (layers *.Cu *.Mask)
-      (net 15 "Tx") (pinfunction "Pin_8") (pintype "passive"))
-    (pad "9" thru_hole oval (at 0.025 6.37) (size 1.7 1.7) (drill 1) (layers *.Cu *.Mask)
-      (net 14 "Rx") (pinfunction "Pin_9") (pintype "passive"))
-    (pad "10" thru_hole oval (at 0.025 8.91) (size 1.7 1.7) (drill 1) (layers *.Cu *.Mask)
+    (pad "8" thru_hole oval (at 0.025 3.83 180) (size 1.7 1.7) (drill 1) (layers *.Cu *.Mask)
+      (net 14 "Rx") (pinfunction "Pin_8") (pintype "passive"))
+    (pad "9" thru_hole oval (at 0.025 6.37 180) (size 1.7 1.7) (drill 1) (layers *.Cu *.Mask)
+      (net 15 "Tx") (pinfunction "Pin_9") (pintype "passive"))
+    (pad "10" thru_hole oval (at 0.025 8.91 180) (size 1.7 1.7) (drill 1) (layers *.Cu *.Mask)
       (net 32 "unconnected-(J1-Pad10)") (pinfunction "Pin_10") (pintype "passive+no_connect"))
-    (pad "11" thru_hole oval (at 0.025 11.45) (size 1.7 1.7) (drill 1) (layers *.Cu *.Mask)
+    (pad "11" thru_hole oval (at 0.025 11.45 180) (size 1.7 1.7) (drill 1) (layers *.Cu *.Mask)
       (net 33 "unconnected-(J1-Pad11)") (pinfunction "Pin_11") (pintype "passive+no_connect"))
-    (pad "12" thru_hole oval (at 0.025 13.99) (size 1.7 1.7) (drill 1) (layers *.Cu *.Mask)
-      (net 34 "unconnected-(J1-Pad12)") (pinfunction "Pin_12") (pintype "passive+no_connect"))
+    (pad "12" thru_hole oval (at 0.025 13.99 180) (size 1.7 1.7) (drill 1) (layers *.Cu *.Mask)
+      (net 34 "GNDA") (pinfunction "Pin_12") (pintype "passive"))
     (model "${KICAD6_3DMODEL_DIR}/Connector_PinSocket_2.54mm.3dshapes/PinSocket_1x12_P2.54mm_Vertical.wrl"
       (offset (xyz 0 0 0))
@@
   (segment (start 164.08 93.58) (end 172.504 93.58) (width 0.5) (layer "F.Cu") (net 2))
   (segment (start 139.9475 86.49) (end 156.99 86.49) (width 0.5) (layer "F.Cu") (net 2))
-  (segment (start 163.063511 120.800489) (end 172.504 111.36) (width 0.5) (layer "F.Cu") (net 14))
-  (segment (start 138.697989 120.197989) (end 139.300489 120.800489) (width 0.5) (layer "F.Cu") (net 14))
-  (segment (start 139.9475 116.97) (end 138.697989 118.219511) (width 0.5) (layer "F.Cu") (net 14))
-  (segment (start 138.697989 118.219511) (end 138.697989 120.197989) (width 0.5) (layer "F.Cu") (net 14))
-  (segment (start 139.300489 120.800489) (end 163.063511 120.800489) (width 0.5) (layer "F.Cu") (net 14))
-  (segment (start 146.277011 113.180489) (end 139.9475 119.51) (width 0.5) (layer "F.Cu") (net 15))
-  (segment (start 168.143511 113.180489) (end 146.277011 113.180489) (width 0.5) (layer "F.Cu") (net 15))
-  (segment (start 172.504 108.82) (end 168.143511 113.180489) (width 0.5) (layer "F.Cu") (net 15))
-  (segment (start 160.2675 106.81) (end 169.434 106.81) (width 0.5) (layer "F.Cu") (net 22))
-  (segment (start 169.434 106.81) (end 172.504 103.74) (width 0.5) (layer "F.Cu") (net 22))
+  (segment (start 170.759489 102.854511) (end 172.454 101.16) (width 0.25) (layer "F.Cu") (net 14))
+  (segment (start 139.772689 120.925489) (end 142.021711 120.925489) (width 0.25) (layer "F.Cu") (net 14))
+  (segment (start 142.021711 120.925489) (end 160.092689 102.854511) (width 0.25) (layer "F.Cu") (net 14))
+  (segment (start 139.9475 116.97) (end 138.822989 118.094511) (width 0.25) (layer "F.Cu") (net 14))
+  (segment (start 138.822989 119.975789) (end 139.772689 120.925489) (width 0.25) (layer "F.Cu") (net 14))
+  (segment (start 160.092689 102.854511) (end 170.759489 102.854511) (width 0.25) (layer "F.Cu") (net 14))
+  (segment (start 138.822989 118.094511) (end 138.822989 119.975789) (width 0.25) (layer "F.Cu") (net 14))
+  (segment (start 171.899489 100.605489) (end 172.454 101.16) (width 0.25) (layer "F.Cu") (net 14))
+  (segment (start 139.9475 119.51) (end 158.852011 100.605489) (width 0.25) (layer "F.Cu") (net 15))
+  (segment (start 170.468511 100.605489) (end 172.454 98.62) (width 0.25) (layer "F.Cu") (net 15))
+  (segment (start 158.852011 100.605489) (end 170.468511 100.605489) (width 0.25) (layer "F.Cu") (net 15))
+  (segment (start 171.884 106.81) (end 172.454 106.24) (width 0.25) (layer "F.Cu") (net 22))
+  (segment (start 160.2675 106.81) (end 171.884 106.81) (width 0.25) (layer "F.Cu") (net 22))
   (zone (net 4) (net_name "GND") (layer "F.Cu") (hatch edge 0.508)
     (connect_pads (clearance 0.508))
